File: kicad/choc/horizon-choc-mini.kicad_pcb (KiCad board)
At the start: 2 copper layers, 216 x 68 mm, 102 parts, among them SW1 SW_Push, SW10 SW_Push, SW11 SW_Push, SW12 SW_Push, SW13 SW_Push, SW14 SW_Push, SW15 SW_Push, SW16 SW_Push, SW17 SW_Push, SW18 SW_Push, SW19 SW_Push, SW2 SW_Push, SW20 SW_Push, SW21 SW_Push, SW22 SW_Push, SW23 SW_Push, SW24 SW_Push, SW25 SW_Push, SW26 SW_Push, SW27 SW_Push, SW28 SW_Push, SW29 SW_Push, SW3 SW_Push, SW30 SW_Push, SW31 SW_Push, SW32 SW_Push, SW33 SW_Push, SW34 SW_Push, SW35 SW_Push, SW36 SW_Push, SW37 SW_Push, SW38 SW_Push, SW39 SW_Push, SW4 SW_Push, SW40 SW_Push, SW41 SW_Push, SW42 SW_Push, SW43 SW_Push, SW44 SW_Push, SW5 SW_Push, SW6 SW_Push, SW7 SW_Push, SW8 SW_Push, SW9 SW_Push, U1 PRO-MICRO

Commit message: Submitting to JLCPCB!
Parts:
- LOGO1: footprint horizon-footprints:Logo_Horizon_Small -> horizon-footprints:bloodborne_moon
- LOGO2: footprint horizon-footprints:Logo_Horizon_H -> horizon-footprints:bloodborne_moon
- moved LOGO2 0.50 mm to (150.0, 88.0)
Routing:
- net ROW2: track 240.7 -> 248.8 mm
- net COL12: track 158.0 -> 162.1 mm
- net COL11: track 138.5 -> 141.9 mm
- net COL10: track 119.5 -> 121.7 mm
- net COL9: track 100.4 -> 101.6 mm
Other:
- board text added: "JLCJLCJLCJLC"
- board text removed: "Black-"
- board text removed: "Red+"
