File: kicad/choc mx spacing/horizon-choc-mini-mx-spacing.kicad_pcb (KiCad board)
At the start: 2 copper layers, 216 x 72 mm, 101 parts, among them SW1 SW_Push, SW10 SW_Push, SW11 SW_Push, SW12 SW_Push, SW13 SW_Push, SW14 SW_Push, SW15 SW_Push, SW16 SW_Push, SW17 SW_Push, SW18 SW_Push, SW19 SW_Push, SW2 SW_Push, SW20 SW_Push, SW21 SW_Push, SW22 SW_Push, SW23 SW_Push, SW24 SW_Push, SW25 SW_Push, SW26 SW_Push, SW27 SW_Push, SW28 SW_Push, SW29 SW_Push, SW3 SW_Push, SW30 SW_Push, SW31 SW_Push, SW32 SW_Push, SW33 SW_Push, SW34 SW_Push, SW35 SW_Push, SW36 SW_Push, SW37 SW_Push, SW38 SW_Push, SW39 SW_Push, SW4 SW_Push, SW40 SW_Push, SW41 SW_Push, SW42 SW_Push, SW43 SW_Push, SW44 SW_Push, SW5 SW_Push, SW6 SW_Push, SW7 SW_Push, SW8 SW_Push, SW9 SW_Push, U3 Nice_Nano_V2

Commit message: - Fix flipped MCU footprint - Fix power switch label
Parts:
- added LOGO1: Logo-Bottom, horizon-footprints:bloodborne_moon, F.Cu at (-111.9, -25.9)
- LOGO2: footprint horizon-footprints:Logo_Horizon_H -> horizon-footprints:bloodborne_moon
- U3: footprint ScottoKeebs_MCU:Nice_Nano_V2 -> ScottoKeebs_MCU:Nice_Nano_V2_Flipped
- moved LOGO2 0.50 mm to (150.0, 87.7)
Connections:
- U3 pad 10: COL4 -> COL9
- U3 pad 11: COL5 -> COL8
- U3 pad 12: COL6 -> COL7
- U3 pad 13: COL7 -> COL6
- U3 pad 14: COL8 -> COL5
- U3 pad 15: COL9 -> COL4
- U3 pad 16: COL10 -> COL3
- U3 pad 17: COL11 -> COL2
- U3 pad 18: unconnected-(U3-D19-Pad18) -> COL1
- U3 pad 19: unconnected-(U3-D20-Pad19) -> COL0
- U3 pad 20: ROW3 -> ROW2
- U3 pad 5: ROW2 -> ROW3
- U3 pad 6: COL0 -> unconnected-(U3-D3-Pad6)
- U3 pad 7: COL1 -> unconnected-(U3-D4-Pad7)
- U3 pad 8: COL2 -> COL11
- U3 pad 9: COL3 -> COL10
Routing:
- net RESET: track 30.5 -> 11.5 mm
- net COL6: track 39.4 -> 52.2 mm
- net COL7: track 84.3 -> 93.3 mm
- net COL0: track 164.6 -> 157.4 mm
- net COL8: track 103.3 -> 109.6 mm
- net Net-(BATJ2-Pin_1): track 15.5 -> 20.3 mm, vias 0 -> 1
- net COL4: track 86.4 -> 90.2 mm
- net COL9: track 122.4 -> 125.9 mm
- net ROW0: track 225.0 -> 221.8 mm
- net COL3: track 105.4 -> 108.5 mm
- net COL1: track 143.5 -> 141.1 mm
- net ROW1: track 242.4 -> 244.4 mm
- net GND: track 43.7 -> 45.4 mm
- net ROW3: track 272.1 -> 273.5 mm
- net COL11: track 160.5 -> 159.5 mm
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